File: esquemasParaBanco/_autosave-esquemasParaBanco.sch (KiCad schematic (older format))
At the start: 237 parts, among them P1 P1, P1 SW_Push, P2 SW_Push

Commit message: added new
Parts:
- added A (x2), B, C, D1, D2: LED, symbol Device:LED
- added BT? (x3): Battery_Cell, symbol Device:Battery_Cell
- added P1, P2: SW_Push, symbol Switch:SW_Push
- added R? (x4): 4Ω, symbol Device:R
- added R? (x2): 6Ω, symbol Device:R
- added R? (x2): 3Ω, symbol Device:R
- added R? (x3): 9Ω, symbol Device:R
- added S1, S2: SW_SPST, symbol Switch:SW_SPST
Connections:
- wire segments 441 -> 491
Other:
- moved on the sheet: A, B, C
