File: esquemasParaBanco/esquemasParaBanco.sch (KiCad schematic (older format))
At the start: 212 parts, among them P1 P1, P1 SW_Push, P2 SW_Push

Commit message: added new
Parts:
- added A (x5), B (x4), C (x4), D, D1, D2, E: LED, symbol Device:LED
- added BT? (x6): Battery_Cell, symbol Device:Battery_Cell
- added P1, P2: SW_Push, symbol Switch:SW_Push
- added R? (x3): 2Ω, symbol Device:R
- added R?: 6Ω, symbol Device:R
- added R?: 3Ω, symbol Device:R
- added R? (x2): 4Ω, symbol Device:R
- added S1, S2: SW_SPST, symbol Switch:SW_SPST
Connections:
- wire segments 372 -> 457
Other:
- note added: "DÍODOS"
- note added: "RESIS EQ"

Commit message: added new
Parts:
- added A (x5), B (x5), C (x4), D (x2): LED, symbol Device:LED
- added BT? (x6): Battery_Cell, symbol Device:Battery_Cell
- added P: SW_Push, symbol Switch:SW_Push
- added R? (x4): 4Ω, symbol Device:R
- added R? (x2): 6Ω, symbol Device:R
- added R? (x2): 3Ω, symbol Device:R
- added R? (x3): 9Ω, symbol Device:R
- added R? (x3): 2Ω, symbol Device:R
Connections:
- wire segments 457 -> 552
